Commit message: Add inertia matrix to urdf

File: src/tartinator/urdf/tartinator.urdf.xacro (robot description, xacro)
@@ -21,4 +21,9 @@
             </geometry>
         </collision>
+        <inertial>
+            <origin xyz="0 0 0" rpy="1.57 0 0"/>
+            <mass value="4"/>
+            <inertia ixx="0.049" ixy="0.0" ixz="0.0" iyy="0.062" iyz="0.0" izz="0.042"/>
+        </inertial>
     </link>
     <link name="left_wheel">
@@ -31,9 +36,14 @@
         </visual>
         <collision>
-            <origin xyz="0 0 -0.02005" rpy="1.57 0 0"/>
+            <origin xyz="-0.098 0 -0.02005" rpy="1.57 0 0"/>
             <geometry>
                 <mesh filename="file://$(find tartinator)/meshes/tartinator_roue_gauche.stl" scale="0.001 0.001 0.001"/>
             </geometry>
         </collision>
+        <inertial>
+            <origin xyz="-0.098 0 -0.02005" rpy="1.57 0 0"/>
+            <mass value="0.2"/>
+            <inertia ixx="0.0001024" ixy="0.0" ixz="0.0" iyy="0.0000629041666667" iyz="0.0" izz="0.0000629041666667"/>
+        </inertial>
     </link>
     <link name="right_wheel">
@@ -46,9 +56,14 @@
         </visual>
         <collision>
-            <origin xyz="0 0 -0.02005" rpy="1.57 0 0"/>
+            <origin xyz="0.098 0 -0.02005" rpy="1.57 0 0"/>
             <geometry>
                 <mesh filename="file://$(find tartinator)/meshes/tartinator_roue_droite.stl" scale="0.001 0.001 0.001"/>
             </geometry>
         </collision>
+        <inertial>
+            <origin xyz="0.098 0 -0.02005" rpy="1.57 0 0"/>
+            <mass value="0.2"/>
+            <inertia ixx="0.0001024" ixy="0.0" ixz="0.0" iyy="0.0000629041666667" iyz="0.0" izz="0.0001024"/>
+        </inertial>
     </link>
     <link name="lidar">
@@ -61,10 +76,16 @@
         </visual>
         <collision>
-            <origin xyz="0 0 0" rpy="1.57 0 0"/>
+            <origin xyz="0 -0.027 0.2919" rpy="1.57 0 0"/>
             <geometry>
                 <mesh filename="file://$(find tartinator)/meshes/tartinator_lidar_urg04lx.stl" scale="0.001 0.001 0.001"/>
             </geometry>
         </collision>
+        <inertial>
+            <origin xyz="0 -0.027 0.2919" rpy="1.57 0 0"/>
+            <mass value="0.4"/>
+            <inertia ixx="0.000251366666667" ixy="0.0" ixz="0.0" iyy="0.000251366666667" iyz="0.0" izz="0.000166666666667"/>
+        </inertial>
     </link>
+    <link name="test_link"></link>
     <!-- Joint -->
     <!-- Base joint -->
@@ -91,3 +112,8 @@
         <child link="lidar"/>
     </joint>
+    <joint name="test_joint" type="fixed">
+        <origin xyz="0.098 0 0" rpy="0 0 0"/>
+        <parent link="right_wheel"/>
+        <child link="test_link"/>
+    </joint>
 </robot>
